File: Hardware/Gordak_Pace.kicad_sch (KiCad schematic)
At the start: 49 parts, among them J1 Screw_Terminal_01x01, J10 Screw_Terminal_01x01, J11 Screw_Terminal_01x01, J12 Screw_Terminal_01x01, J13 Screw_Terminal_01x01, J14 DIN-6, J15 DIN-6, J2 Screw_Terminal_01x01, J4 Screw_Terminal_01x01, J5 Screw_Terminal_01x01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

Commit message: Add files via upload
Other:
- note added: "PTC +"
- note added: "PTC -"
- note added: "Pace MBT 250 rework station with a Gordak handpiece and Arduino by Fodor Tibor https://www.youtube.com/watch?v=LTK6tuzxlCQ Schematic: Greenonline/Gr33nonline"
- note added: "Together, these resistors are 200R in total"
- note removed: "Pace MBT 250 rework station with a Gordak handpiece and Arduino by Fodor Tibor https://www.youtube.com/watch?v=LTK6tuzxlCQ Schematic: M.G. Jenkins (Greenonline/Gr33nonline)"
Changed lines of the file:
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@@
     (effects (font (size 1.27 1.27)) (justify left bottom))
   )
-  (text "Thermocouple -" (at 262.89 120.65 0)
+  (text "PTC -" (at 262.89 120.65 0)
     (effects (font (size 1.27 1.27)) (justify left bottom))
   )
@@
     (effects (font (size 1.27 1.27)) (justify left bottom))
   )
-  (text "Pace MBT 250 rework station with a Gordak handpiece and Arduino by Fodor Tibor\n\nhttps://www.youtube.com/watch?v=LTK6tuzxlCQ\n\nSchematic: M.G. Jenkins (Greenonline/Gr33nonline)"
+  (text "Pace MBT 250 rework station with a Gordak handpiece and Arduino by Fodor Tibor\n\nhttps://www.youtube.com/watch?v=LTK6tuzxlCQ\n\nSchematic: Greenonline/Gr33nonline"
     (at 180.34 180.34 0)
     (effects (font (size 1.27 1.27)) (justify left bottom))
@@
     (effects (font (size 1.27 1.27)) (justify left bottom))
   )
-  (text "Thermocouple +" (at 262.89 113.03 0)
+  (text "PTC +" (at 262.89 113.03 0)
     (effects (font (size 1.27 1.27)) (justify left bottom))
   )
@@
     (effects (font (size 1.27 1.27)) (justify left bottom))
   )
+  (text "Together, these resistors are 200R in total" (at 109.22 39.37 0)
+    (effects (font (size 1.27 1.27)) (justify left bottom))
+  )

Commit message: Add files via upload
Parts:
- removed J14: DIN-6, symbol Connector:DIN-6
- added J14: DIN-5, symbol Connector:DIN-5
Connections:
- net at J7.1 (Pin_1): now also J14.2
- net at J6.1 (Pin_1): now also J14.1
- net at J4.1 (Pin_1): now also J14.5
- net at J5.1 (Pin_1): now also J14.4
